File: Plaquinha.kicad_sch (KiCad schematic)
At the start: 33 parts, among them J1 Screw_Terminal_01x02, J10 Conn_01x15_Socket, J11 Conn_01x15_Socket, J12 Conn_01x06_Socket, J2 Conn_01x10_Socket, J3 Conn_01x10_Socket, J4 Conn_01x06_Socket, J5 Conn_01x04_Socket, J6 Conn_01x04_Socket, J8 Conn_01x03_Socket, J9 Conn_01x03_Socket, U1 L7805, U10 TA6586, U3 TA6586, U5 L7805, U9 ESP32-DEVKIT-V1

Commit message: Refazendo a cagada
Parts:
- BZ1: footprint (none) -> Buzzer_Beeper:Buzzer_TDK_PS1240P02BT_D12.2mm_H6.5mm
- C1: footprint (none) -> Capacitor_THT:C_Disc_D5.0mm_W2.5mm_P2.50mm
- C4, C5, C6: footprint (none) -> Capacitor_THT:C_Disc_D5.0mm_W2.5mm_P5.00mm
- C7, C8: footprint Capacitor_THT:C_Radial_D6.3mm_H5.0mm_P2.50mm -> Capacitor_THT:C_Disc_D5.0mm_W2.5mm_P5.00mm
- D1: footprint (none) -> Diode_THT:D_A-405_P7.62mm_Horizontal
- D2, D3: footprint (none) -> LED_THT:LED_D3.0mm
- J12, J4: footprint Connector_PinHeader_2.54mm:PinHeader_1x06_P2.54mm_Vertical -> Connector_JST:JST_EH_B6B-EH-A_1x06_P2.50mm_Vertical
- R1, R3: footprint (none) -> Resistor_THT:R_Axial_DIN0204_L3.6mm_D1.6mm_P5.08mm_Horizontal
- U9: footprint ESPFootprint:Module_ESP32_DEVKIT_V1 -> ESPFootprint:MODULE_ESP32_DEVKIT_V1
Connections:
- net D32: now also U9.21 (D32)
- net D33: now also BZ1.1 (+), U9.22 (D33)
- net D34: now also U9.19 (D34)
- net D35: now also U9.20 (D35)
- net ECHO: now also U9.6 (RX2); no longer U9.23 (D25)
- net EN: now also U9.16 (EN)
- net GND: now also U9.29 (GND__1)
- net TRIG: now also U9.7 (TX2); no longer U9.24 (D26)
- net VN: now also U9.18 (VN)
- net VP: now also U9.17 (VP)
